File: RTC-Kello/RTC-Kello v1.kicad_pcb (KiCad board)
At the start: 2 copper layers, 114.3 x 38.1 mm, 34 parts, among them J1 Screw_Terminal_1x02, J2 CONN_01X06, J3 CONN_01X04, J4 CONN_02X05, J5 CONN_01X02, J6 CONN_01X02, Q1 2N2219, Q2 2N2219, Q3 2N2219, Q4 2N2219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

Commit message: PCB send to OSH Park
Routing:
- added copper zone on B.Cu, net GND
- added copper zone on F.Cu, net GND
Other:
- board text added: "RTC Clock v1.0"
Changed lines of the file:
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@@
     (area 36.45 40.48 185.800001 104.3525)
     (thickness 1.6)
-    (drawings 23)
+    (drawings 24)
     (tracks 408)
     (zones 0)
@@
     (0 F.Cu signal)
     (31 B.Cu signal)
-    (32 B.Adhes user hide)
-    (33 F.Adhes user hide)
-    (34 B.Paste user hide)
-    (35 F.Paste user hide)
+    (32 B.Adhes user)
+    (33 F.Adhes user)
+    (34 B.Paste user)
+    (35 F.Paste user)
     (36 B.SilkS user)
     (37 F.SilkS user)
-    (38 B.Mask user hide)
+    (38 B.Mask user)
     (39 F.Mask user)
-    (40 Dwgs.User user hide)
-    (41 Cmts.User user hide)
-    (42 Eco1.User user hide)
-    (43 Eco2.User user hide)
+    (40 Dwgs.User user)
+    (41 Cmts.User user)
+    (42 Eco1.User user)
+    (43 Eco2.User user)
     (44 Edge.Cuts user)
-    (45 Margin user hide)
-    (46 B.CrtYd user hide)
-    (47 F.CrtYd user hide)
-    (48 B.Fab user hide)
-    (49 F.Fab user hide)
+    (45 Margin user)
+    (46 B.CrtYd user)
+    (47 F.CrtYd user)
+    (48 B.Fab user)
+    (49 F.Fab user)
   )
   (setup
@@
       (padsonsilk false)
       (subtractmaskfromsilk false)
-      (outputformat 1)
+      (outputformat 4)
       (mirror false)
       (drillshape 0)
@@
       (rotate (xyz 0 0 0))
     )
+  )
+  (gr_text "RTC Clock v1.0" (at 78.74 66.04) (layer F.SilkS)
+    (effects (font (size 1.5 1.5) (thickness 0.3)))
   )
   (gr_text tiny2313 (at 74.676 82.296) (layer F.SilkS)
@@
   (segment (start 57.055001 90.619997) (end 57.055001 93.904999) (width 0.25) (layer B.Cu) (net 45))
   (segment (start 57.055001 93.904999) (end 56.98 93.98) (width 0.25) (layer B.Cu) (net 45))
+  (zone (net 1) (net_name GND) (layer F.Cu) (hatch edge 0.508)
+    (connect_pads (clearance 0.508))
+    (min_thickness 0.254)
+    (fill yes (arc_segments 16) (thermal_gap 0.508) (thermal_bridge_width 0.508))
+    (polygon
+      (pts
+        (xy 165.1 101.6) (xy 165.1 63.5) (xy 50.8 63.5) (xy 50.8 101.6)
+      )
+    )
+  )
+  (zone (net 1) (net_name GND) (layer B.Cu) (hatch edge 0.508)
+    (connect_pads (clearance 0.508))
+    (min_thickness 0.254)
+    (fill yes (arc_segments 16) (thermal_gap 0.508) (thermal_bridge_width 0.508))
+    (polygon
+      (pts
+        (xy 165.1 101.6) (xy 165.1 63.5) (xy 50.8 63.5) (xy 50.8 101.6)
+      )
+    )
+  )
 )
