File: RTC-Kello/RTC-Kello.kicad_pcb (KiCad board)
At the start: 2 copper layers, 114.3 x 38.1 mm, 34 parts, among them J1 Screw_Terminal_1x02, J2 CONN_01X06, J3 CONN_01X04, J4 CONN_02X05, J5 CONN_01X02, J6 CONN_01X02, Q1 2N2219, Q2 2N2219, Q3 2N2219, Q4 2N2219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

Commit message: PCB send to OSH Park
Parts:
- moved C1 6.50 mm to (62.2, 66.0), turned to 180 degrees
Routing:
- net +3V3: track 83.6 -> 182.9 mm, vias 1 -> 2
- net GND: track 30.6 -> 105.6 mm, vias 0 -> 2
- net Net-(AFF4-Pad3): track 0.00 -> 24.1 mm, vias 1 -> 2
- net Net-(AFF3-Pad3): track 10.5 -> 25.7 mm, vias 0 -> 1
- net Net-(C1-Pad1): track 6.50 -> 16.0 mm, vias 0 -> 1
